File: stamp_attach.kicad_pcb (KiCad board)
At the start: 2 copper layers, 88 x 90 mm, 25 parts, among them J1 SA_layer_A, J2 SA_layer_D, J3 test_footprint

Commit message: logo and qr (unfinished)
Other:
- board text removed: "Stamp-Attach"
